Commit message: add vp6242 description

File: robotic_arm/vp6242/vp6246_description/robot/vp6242.urdf (robot description, URDF)
Before this commit: robot ve026a, 8 links, 7 joints
Links:
- removed link link5
- removed link link6
- link base_link: geometry visual box size=0.160 0.160 0.155
- link link0: geometry visual cylinder length=0.125 radius=0.075
- link link1: geometry visual cylinder length=0.210 radius=0.075
- link link2: geometry visual cylinder length=0.075 radius=0.075
- link link3: geometry visual cylinder length=0.202 radius=0.075
Joints:
- removed joint J5
- removed joint J6
- removed joint J7
- added joint JF1: type fixed, parent link2, child link3, origin xyz=0.0 0.0 0.075 rpy=0 0 0
- joint J1: limit lower=-1.39626 upper=1.83259 effort=1000.0 velocity=1.0 -> lower=-2.792526 upper=2.792526 effort=1000.0 velocity=1.0; origin xyz=0.0 0.0 0.0 rpy=0 0 0 -> xyz=0.0 0.0 0.155 rpy=0 0 0
- joint J2: limit lower=-0.61086 upper=1.57075 effort=1000.0 velocity=1.0 -> lower=-2.094394 upper=2.094394 effort=1000.0 velocity=1.0; origin xyz=0.0 0.0 0.130 rpy=0 0 0 -> xyz=0.0 0.0 0.125 rpy=0 0 0
- joint J3: limit lower=-1.30899 upper=2.35619 effort=1000.0 velocity=1.0 -> lower=0.331612 upper=2.792526 effort=1000.0 velocity=1.0; origin xyz=0.0 0.0 0.100 rpy=0 0 0 -> xyz=0.0 0.0 0.210 rpy=0 0 0
- joint J4: axis 0 0 1 -> 0 1 0; child link3 -> link4; limit lower=-2.44346 upper=2.44346 effort=1000.0 velocity=1.0 -> lower=-1.57075 upper=1.83259 effort=1000.0 velocity=1.0; origin xyz=0.0 0.0 0.020 rpy=0 0 0 -> xyz=0.0 0.0 0.070 rpy=0 0 0; parent link2 -> link3
