Commit message: - add IK - add simulate

File: robotic_arm/ve026e/ve026a_description/robot/ve026a.urdf (robot description, URDF)
Before this commit: robot ve026a, 10 links, 9 joints
Links:
- removed link gripper_left
- removed link gripper_right
Joints:
- removed joint J7_left
- removed joint J7_right

Commit message: - update ve026a.urdf and planning model  - update vp6242.urdf and add planning model

File: robotic_arm/ve026e/ve026a_description/robot/ve026a.urdf (robot description, URDF)
Before this commit: robot ve026a, 8 links, 7 joints
Joints:
- joint J7: type revolute -> fixed

File: robotic_arm/vp6242/vp6246_description/robot/vp6242.urdf (robot description, URDF)
Before this commit: robot vp6242, 6 links, 5 joints
Links:
- added link link5; visual cylinder length=0.010 radius=0.0325
- link base_link: geometry visual cylinder length=0.125 radius=0.08
- link link0: geometry visual cylinder length=0.125 radius=0.03
- link link1: geometry visual cylinder length=0.210 radius=0.03
- link link2: geometry visual cylinder length=0.075 radius=0.03
- link link3: geometry visual cylinder length=0.311 radius=0.03
- link link4: geometry visual cylinder length=0.060 radius=0.0325
Joints:
- removed joint JF1
- added joint J5: type revolute, parent link3, child link4, origin xyz=0.210 0.0 0.0 rpy=0 0 0, axis 0 1 0, limit lower=-2.094394 upper=2.094394 effort=1000.0 velocity=1.0
- added joint J6: type revolute, parent link4, child link5, origin xyz=0.06 0.0 0.0 rpy=0 0 0, axis 1 0 0, limit lower=-2.094394 upper=2.094394 effort=1000.0 velocity=1.0
- joint J3: limit lower=0.331612 upper=2.792526 effort=1000.0 velocity=1.0 -> lower=-1.239183 upper=1.221730 effort=1000.0 velocity=1.0
- joint J4: axis 0 1 0 -> 1 0 0; child link4 -> link3; limit lower=-1.57075 upper=1.83259 effort=1000.0 velocity=1.0 -> lower=-2.792526 upper=2.792526 effort=1000.0 velocity=1.0; origin xyz=0.0 0.0 0.070 rpy=0 0 0 -> xyz=0.0 0.0 0.075 rpy=0 0 0; parent link3 -> link2

Commit message: scene warehouse is working!

File: robotic_arm/ve026e/ve026a_description/robot/ve026a.urdf (robot description, URDF)
Before this commit: robot ve026a, 8 links, 7 joints
Links:
- link base_link: mass None -> 0.1; geometry collision box size=0.079 0.079 0.006; visual box size=0.079 0.079 0.006
- link link0: mass None -> 0.1; geometry collision cylinder length=0.130 radius=0.035; visual cylinder length=0.130 radius=0.035
- link link1: mass None -> 0.1; geometry collision box size=0.040 0.050 0.100; visual box size=0.040 0.050 0.100
- link link2: mass None -> 0.1; geometry collision box size=0.040 0.030 0.020; visual box size=0.040 0.030 0.020
- link link3: mass None -> 0.1; geometry collision box size=0.030 0.050 0.070; visual box size=0.030 0.050 0.070
- link link4: mass None -> 0.1; geometry collision box size=0.040 0.030 0.020; visual box size=0.040 0.030 0.020
- link link5: mass None -> 0.1; geometry collision box size=0.050 0.030 0.068; visual box size=0.050 0.030 0.068
- link link6: mass None -> 0.1; geometry collision box size=0.050 0.030 0.010; visual box size=0.050 0.030 0.010
Joints:
- joint J1: limit lower=-1.39626 upper=1.83259 effort=1000.0 velocity=1.0 -> lower=-1.39626 upper=1.83259 effort=1000.0 velocity=3.0
- joint J2: limit lower=-0.61086 upper=1.57075 effort=1000.0 velocity=1.0 -> lower=-0.61086 upper=1.57075 effort=1000.0 velocity=3.0
- joint J3: limit lower=-1.30899 upper=2.35619 effort=1000.0 velocity=1.0 -> lower=-1.30899 upper=2.35619 effort=1000.0 velocity=3.0
- joint J4: limit lower=-2.44346 upper=2.44346 effort=1000.0 velocity=1.0 -> lower=-2.44346 upper=2.44346 effort=1000.0 velocity=3.0
- joint J5: limit lower=-1.57075 upper=1.83259 effort=1000.0 velocity=1.0 -> lower=-1.57075 upper=1.83259 effort=1000.0 velocity=3.0
- joint J6: limit lower=-2.44346 upper=2.44346 effort=1000.0 velocity=1.0 -> lower=-2.44346 upper=2.44346 effort=1000.0 velocity=3.0
- joint J7: limit lower=-1.30899 upper=0.43633 effort=1000.0 velocity=1.0 -> lower=-1.30899 upper=0.43633 effort=1000.0 velocity=3.0

Commit message: updated ve026a.urdf with stl model

File: robotic_arm/ve026e/ve026a_description/robot/ve026a.urdf (robot description, URDF)
Before this commit: robot ve026a, 8 links, 7 joints
Links:
- link base_link: geometry collision box size=0.079 0.079 0.006; visual mesh filename=package://ve026a_description/robot/base.stl scale=1 1 1
- link link0: geometry collision cylinder length=0.130 radius=0.035; visual mesh filename=package://ve026a_description/robot/l0.stl scale=1 1 1
- link link1: geometry collision box size=0.040 0.050 0.100; visual mesh filename=package://ve026a_description/robot/l1.stl scale=1 1 1
- link link2: geometry collision box size=0.040 0.050 0.100; visual mesh filename=package://ve026a_description/robot/l2.stl scale=1 1 1
- link link3: geometry collision box size=0.040 0.030 0.020; visual mesh filename=package://ve026a_description/robot/l3.stl scale=1 1 1
- link link4: geometry collision box size=0.030 0.050 0.070; visual mesh filename=package://ve026a_description/robot/l4.stl scale=1 1 1
- link link5: geometry collision box size=0.040 0.030 0.020; visual mesh filename=package://ve026a_description/robot/l5.stl scale=1 1 1
- link link6: geometry collision box size=0.050 0.030 0.068; visual mesh filename=package://ve026a_description/robot/l6.stl scale=1 1 1
Joints:
- removed joint J7
- added joint J0: type fixed, parent base_link, child link0, origin xyz=0.0 0.0 0.0 rpy=0 0 0, axis 0 0 1
- joint J1: child link0 -> link1; parent base_link -> link0
- joint J2: child link1 -> link2; parent link0 -> link1
- joint J3: child link2 -> link3; parent link1 -> link2
- joint J4: child link3 -> link4; origin xyz=0.0 0.0 0.020 rpy=0 0 0 -> xyz=0.0 0.0 0.018 rpy=0 0 0; parent link2 -> link3
- joint J5: child link4 -> link5; origin xyz=0.0 0.0 0.070 rpy=0 0 0 -> xyz=0.0 0.0 0.075 rpy=0 0 0; parent link3 -> link4
- joint J6: child link5 -> link6; origin xyz=0.0 0.0 0.020 rpy=0 0 0 -> xyz=0.0 0.0 0.018 rpy=0 0 0; parent link4 -> link5

Commit message: - reduced robot mesh size  - updated planning scene  - updated planning warehouse

File: robotic_arm/ve026e/ve026a_description/robot/ve026a.urdf (robot description, URDF)
Before this commit: robot ve026a, 8 links, 7 joints
Links:
- added link link7, mass 0.1; visual cylinder length=0.010 radius=0.01
- link base_link: geometry visual mesh filename=package://ve026a_description/robot/base.stl scale=1 1 1
- link link0: geometry visual mesh filename=package://ve026a_description/robot/l0.stl scale=1 1 1
- link link1: geometry visual mesh filename=package://ve026a_description/robot/l1.stl scale=1 1 1
- link link2: geometry visual mesh filename=package://ve026a_description/robot/l2.stl scale=1 1 1
- link link3: geometry visual mesh filename=package://ve026a_description/robot/l3.stl scale=1 1 1
- link link4: geometry visual mesh filename=package://ve026a_description/robot/l4.stl scale=1 1 1
- link link5: geometry visual mesh filename=package://ve026a_description/robot/l5.stl scale=1 1 1
- link link6: geometry visual mesh filename=package://ve026a_description/robot/l6.stl scale=1 1 1
Joints:
- added joint J7: type revolute, parent link6, child link7, origin xyz=0.0 0.0 0.068 rpy=0 0 0, axis 0 0 1, limit lower=-1.30899 upper=0.43633 effort=1000.0 velocity=3.0
