Commit message: - added vp6242 model  - updated planning scene  - added planning scene warehouse

File: robotic_arm/vp6242/vp6242_description/robot/vp6242.urdf (robot description, URDF)
Before this commit: robot vp6242, 7 links, 6 joints
Links:
- link base_link: geometry visual mesh filename=package://vp6242_description/robot/base.stl scale=0.001 0.001 0.001
- link link0: geometry visual mesh filename=package://vp6242_description/robot/l0.stl scale=0.001 0.001 0.001
- link link1: geometry visual mesh filename=package://vp6242_description/robot/l1.stl scale=0.001 0.001 0.001
- link link2: geometry visual mesh filename=package://vp6242_description/robot/l2.stl scale=0.001 0.001 0.001
- link link3: geometry visual mesh filename=package://vp6242_description/robot/l3.stl scale=0.001 0.001 0.001
- link link4: geometry visual mesh filename=package://vp6242_description/robot/l4.stl scale=0.001 0.001 0.001
- link link5: geometry visual cylinder length=0.010 radius=0.02
Joints:
- joint J4: origin xyz=0.0 0.0 0.075 rpy=0 0 0 -> xyz=0.079729 0.0 0.075 rpy=0 0 0
- joint J5: origin xyz=0.210 0.0 0.0 rpy=0 0 0 -> xyz=0.130271 0.0 0.0 rpy=0 0 0
