Commit message: - learning boost asio  - will use it in ve026a_teleop.cpp

File: robotic_arm/ve026a/ve026a_description/robot/ve026a.urdf (robot description, URDF)
Before this commit: robot ve026a, 9 links, 8 joints
Joints:
- joint J1: limit lower=-1.39626 upper=1.83259 effort=1000.0 velocity=3.0 -> lower=-1.39626 upper=1.83259 effort=1000.0 velocity=6.0
- joint J2: limit lower=-0.61086 upper=1.57075 effort=1000.0 velocity=3.0 -> lower=-0.61086 upper=1.57075 effort=1000.0 velocity=6.0
- joint J3: limit lower=-1.30899 upper=2.35619 effort=1000.0 velocity=3.0 -> lower=-1.30899 upper=2.35619 effort=1000.0 velocity=6.0
- joint J4: limit lower=-2.44346 upper=2.44346 effort=1000.0 velocity=3.0 -> lower=-2.44346 upper=2.44346 effort=1000.0 velocity=6.0
- joint J5: limit lower=-1.57075 upper=1.83259 effort=1000.0 velocity=3.0 -> lower=-1.57075 upper=1.83259 effort=1000.0 velocity=6.0
- joint J6: limit lower=-2.44346 upper=2.44346 effort=1000.0 velocity=3.0 -> lower=-2.44346 upper=2.44346 effort=1000.0 velocity=6.0
- joint J7: limit lower=-1.30899 upper=0.43633 effort=1000.0 velocity=3.0 -> lower=-1.30899 upper=0.43633 effort=1000.0 velocity=6.0

Commit message: added simple client-server teleop via TCP/IP

File: robotic_arm/ve026a/ve026a_description/robot/ve026a.urdf (robot description, URDF)
Before this commit: robot ve026a, 9 links, 8 joints
Joints:
- joint J1: limit lower=-1.39626 upper=1.83259 effort=1000.0 velocity=6.0 -> lower=-1.39626 upper=1.83259 effort=1000.0 velocity=3.0
- joint J2: limit lower=-0.61086 upper=1.57075 effort=1000.0 velocity=6.0 -> lower=-0.61086 upper=1.57075 effort=1000.0 velocity=3.0
- joint J3: limit lower=-1.30899 upper=2.35619 effort=1000.0 velocity=6.0 -> lower=-1.30899 upper=2.35619 effort=1000.0 velocity=3.0
- joint J4: limit lower=-2.44346 upper=2.44346 effort=1000.0 velocity=6.0 -> lower=-2.44346 upper=2.44346 effort=1000.0 velocity=3.0
- joint J5: limit lower=-1.57075 upper=1.83259 effort=1000.0 velocity=6.0 -> lower=-1.57075 upper=1.83259 effort=1000.0 velocity=3.0
- joint J6: limit lower=-2.44346 upper=2.44346 effort=1000.0 velocity=6.0 -> lower=-2.44346 upper=2.44346 effort=1000.0 velocity=3.0
- joint J7: limit lower=-1.30899 upper=0.43633 effort=1000.0 velocity=6.0 -> lower=-0.63633 upper=0.43633 effort=1000.0 velocity=3.0
