Commit message: - planning scene warehouse is working  - all joint information in ROS will respect to URDF setting    - e.g. J3 of VP6424

File: denso/vp6242/vp6242_description/robot/vp6242.urdf (robot description, URDF)
Before this commit: robot vp6242, 7 links, 6 joints
Joints:
- joint J1: limit lower=-2.792526 upper=2.792526 effort=1000.0 velocity=1.0 -> lower=-2.792526 upper=2.792526 effort=1000.0 velocity=0.1
- joint J2: limit lower=-2.094394 upper=2.094394 effort=1000.0 velocity=1.0 -> lower=-2.094394 upper=2.094394 effort=1000.0 velocity=0.1
- joint J3: limit lower=-1.239183 upper=1.221730 effort=1000.0 velocity=1.0 -> lower=-1.239183 upper=1.221730 effort=1000.0 velocity=0.1
- joint J4: limit lower=-2.792526 upper=2.792526 effort=1000.0 velocity=1.0 -> lower=-2.792526 upper=2.792526 effort=1000.0 velocity=0.1
- joint J5: limit lower=-2.094394 upper=2.094394 effort=1000.0 velocity=1.0 -> lower=-2.094394 upper=2.094394 effort=1000.0 velocity=0.1
- joint J6: limit lower=-2.094394 upper=2.094394 effort=1000.0 velocity=1.0 -> lower=-2.094394 upper=2.094394 effort=1000.0 velocity=0.1

Commit message: corrected VP6242 URDF (J6 position) added real robot launch file for prw test

File: denso/vp6242/vp6242_description/robot/vp6242.urdf (robot description, URDF)
Before this commit: robot vp6242, 7 links, 6 joints
Joints:
- joint J6: origin xyz=0.06 0.0 0.0 rpy=0 0 0 -> xyz=0.07 0.0 0.0 rpy=0 0 0

Commit message: corrected vp6242 urdf

File: denso/vp6242/vp6242_description/robot/vp6242.urdf (robot description, URDF)
Before this commit: robot vp6242, 7 links, 6 joints
Joints:
- joint J6: limit lower=-2.094394 upper=2.094394 effort=1000.0 velocity=0.1 -> lower=-6.283185 upper=6.283185 effort=1000.0 velocity=0.1

Commit message: a lot of updates
trajectory filter has problem with smalll displacement path (use a lot of time)

File: denso/vp6242/vp6242_description/robot/vp6242.urdf (robot description, URDF)
Before this commit: robot vp6242, 7 links, 6 joints
Joints:
- joint J1: limit lower=-2.792526 upper=2.792526 effort=1000.0 velocity=0.1 -> lower=-2.792526 upper=2.792526 effort=1000.0 velocity=1.0
- joint J2: limit lower=-2.094394 upper=2.094394 effort=1000.0 velocity=0.1 -> lower=-2.094394 upper=2.094394 effort=1000.0 velocity=1.0
- joint J3: limit lower=-1.239183 upper=1.221730 effort=1000.0 velocity=0.1 -> lower=-1.239183 upper=1.221730 effort=1000.0 velocity=1.0
- joint J4: limit lower=-2.792526 upper=2.792526 effort=1000.0 velocity=0.1 -> lower=-2.792526 upper=2.792526 effort=1000.0 velocity=1.0
- joint J5: limit lower=-2.094394 upper=2.094394 effort=1000.0 velocity=0.1 -> lower=-2.094394 upper=2.094394 effort=1000.0 velocity=1.0
- joint J6: limit lower=-6.283185 upper=6.283185 effort=1000.0 velocity=0.1 -> lower=-6.283185 upper=6.283185 effort=1000.0 velocity=1.0

Commit message: arm move is working

File: denso/vp6242/vp6242_description/robot/vp6242.urdf (robot description, URDF)
Before this commit: robot vp6242, 7 links, 6 joints
Joints:
- joint J1: limit lower=-2.792526 upper=2.792526 effort=1000.0 velocity=1.0 -> lower=-2.792526 upper=2.792526 effort=1000.0 velocity=2.0
- joint J2: limit lower=-2.094394 upper=2.094394 effort=1000.0 velocity=1.0 -> lower=-2.094394 upper=2.094394 effort=1000.0 velocity=2.0
- joint J3: limit lower=-1.239183 upper=1.221730 effort=1000.0 velocity=1.0 -> lower=-1.239183 upper=1.221730 effort=1000.0 velocity=2.0
- joint J4: limit lower=-2.792526 upper=2.792526 effort=1000.0 velocity=1.0 -> lower=-2.792526 upper=2.792526 effort=1000.0 velocity=2.0
- joint J5: limit lower=-2.094394 upper=2.094394 effort=1000.0 velocity=1.0 -> lower=-2.094394 upper=2.094394 effort=1000.0 velocity=2.0
- joint J6: limit lower=-6.283185 upper=6.283185 effort=1000.0 velocity=1.0 -> lower=-6.283185 upper=6.283185 effort=1000.0 velocity=2.0

Commit message: different timeout for filter

File: denso/vp6242/vp6242_description/robot/vp6242.urdf (robot description, URDF)
Before this commit: robot vp6242, 7 links, 6 joints
Joints:
- joint J6: limit lower=-6.283185 upper=6.283185 effort=1000.0 velocity=2.0 -> lower=-3.141592 upper=3.141592 effort=1000.0 velocity=2.0

Commit message: disp.trajectory_bad_point_ -1 -24 GOAL_CONSTRAINTS_VIOLATED???

File: denso/vp6242/vp6242_description/robot/vp6242.urdf (robot description, URDF)
Before this commit: robot vp6242, 7 links, 6 joints
Joints:
- joint J6: limit lower=-3.141592 upper=3.141592 effort=1000.0 velocity=2.0 -> lower=-6.283185 upper=6.283185 effort=1000.0 velocity=2.0

Commit message: updated STL

File: denso/vp6242/vp6242_description/robot/vp6242.urdf (robot description, URDF)
Before this commit: robot vp6242, 7 links, 6 joints
Links:
- link base_link: geometry collision mesh filename=package://vp6242_description/robot/base_collision.stl scale=0.001 0.001 0.001; visual mesh filename=package://vp6242_description/robot/base.stl scale=0.001 0.001 0.001
- link link0: geometry collision mesh filename=package://vp6242_description/robot/l0_collision.stl scale=0.001 0.001 0.001; visual mesh filename=package://vp6242_description/robot/l0.stl scale=0.001 0.001 0.001
- link link1: geometry collision mesh filename=package://vp6242_description/robot/l1_collision.stl scale=0.001 0.001 0.001; visual mesh filename=package://vp6242_description/robot/l1.stl scale=0.001 0.001 0.001
- link link2: geometry collision mesh filename=package://vp6242_description/robot/l2_collision.stl scale=0.001 0.001 0.001; visual mesh filename=package://vp6242_description/robot/l2.stl scale=0.001 0.001 0.001
- link link3: geometry collision mesh filename=package://vp6242_description/robot/l3_collision.stl scale=0.001 0.001 0.001; visual mesh filename=package://vp6242_description/robot/l3.stl scale=0.001 0.001 0.001
- link link4: geometry collision mesh filename=package://vp6242_description/robot/l4_collision.stl scale=0.001 0.001 0.001; visual mesh filename=package://vp6242_description/robot/l4.stl scale=0.001 0.001 0.001
