Commit message: VE026A controller is working

File: robots/denso/ve026a_description/robot/ve026a.urdf (robot description, URDF)
Before this commit: robot ve026a, 9 links, 8 joints
Links:
- removed link link6
- removed link link7
- added link gripper_left; visual box size=0.020 0.002 0.030
- added link gripper_right; visual box size=0.020 0.002 0.030
- link base_link: mass 0.1 -> None; geometry visual cylinder length=0.130 radius=0.035
- link link0: mass 0.1 -> None; geometry visual box size=0.01 0.01 0.01
- link link1: mass 0.1 -> None; geometry visual box size=0.03 0.05 0.1
- link link2: mass 0.1 -> None; geometry visual box size=0.01 0.01 0.01
- link link3: mass 0.1 -> None; geometry visual box size=0.05 0.05 0.09
- link link4: mass 0.1 -> None; geometry visual box size=0.05 0.03 0.088
- link link5: mass 0.1 -> None; geometry visual cylinder length=0.005 radius=0.005
Joints:
- removed joint J0
- removed joint J7
- added joint J7_left: type prismatic, parent link5, child gripper_left, origin xyz=0.0 0.0 0.0 rpy=0 0 0, axis 0 1 0, limit lower=0.013 upper=0.0215 effort=1000.0 velocity=1.0
- added joint J7_right: type prismatic, parent link5, child gripper_right, origin xyz=0.0 0.0 0.0 rpy=0 0 0, axis 0 1 0, limit lower=-0.013 upper=-0.0215 effort=1000.0 velocity=1.0
- joint J1: child link1 -> link0; limit lower=-1.39626 upper=1.83259 effort=1000.0 velocity=3.0 -> lower=-1.39626 upper=1.83259 effort=1000.0 velocity=1.0; origin xyz=0.0 0.0 0.0 rpy=0 0 0 -> xyz=0.0 0.0 0.130 rpy=0 0 0; parent link0 -> base_link
- joint J2: child link2 -> link1; limit lower=-0.61086 upper=1.57075 effort=1000.0 velocity=3.0 -> lower=-0.61086 upper=1.57075 effort=1000.0 velocity=1.0; origin xyz=0.0 0.0 0.130 rpy=0 0 0 -> xyz=0.0 0.0 0.0 rpy=0 0 0; parent link1 -> link0
- joint J3: child link3 -> link2; limit lower=-1.30899 upper=2.35619 effort=1000.0 velocity=3.0 -> lower=-1.30899 upper=2.35619 effort=1000.0 velocity=1.0; parent link2 -> link1
- joint J4: child link4 -> link3; limit lower=-2.44346 upper=2.44346 effort=1000.0 velocity=3.0 -> lower=-2.44346 upper=2.44346 effort=1000.0 velocity=1.0; origin xyz=0.0 0.0 0.018 rpy=0 0 0 -> xyz=0.0 0.0 0.0 rpy=0 0 0; parent link3 -> link2
- joint J5: child link5 -> link4; limit lower=-1.57075 upper=1.83259 effort=1000.0 velocity=3.0 -> lower=-1.57075 upper=1.83259 effort=1000.0 velocity=1.0; origin xyz=0.0 0.0 0.075 rpy=0 0 0 -> xyz=0.0 0.0 0.090 rpy=0 0 0; parent link4 -> link3
- joint J6: child link6 -> link5; limit lower=-2.44346 upper=2.44346 effort=1000.0 velocity=3.0 -> lower=-2.44346 upper=2.44346 effort=1000.0 velocity=1.0; origin xyz=0.0 0.0 0.018 rpy=0 0 0 -> xyz=0.0 0.0 0.088 rpy=0 0 0; parent link5 -> link4
