Commit message: added vp6242 xacro added vp6242 arm navigation

File: robots/denso/vp6242_description/robot/vp6242.urdf (robot description, URDF)
Before this commit: robot vp6242, 7 links, 6 joints
Links:
- link link5: geometry visual cylinder length=0.010 radius=0.021
Joints:
- joint J1: limit lower=-2.792526 upper=2.792526 effort=1000.0 velocity=2.0 -> lower=-2.792526 upper=2.792526 effort=1000.0 velocity=1.0
- joint J2: limit lower=-2.094394 upper=2.094394 effort=1000.0 velocity=2.0 -> lower=-2.094394 upper=2.094394 effort=1000.0 velocity=1.0
- joint J3: limit lower=-1.239183 upper=1.221730 effort=1000.0 velocity=2.0 -> lower=0.331612 upper=2.792526 effort=1000.0 velocity=1.0
- joint J4: limit lower=-2.792526 upper=2.792526 effort=1000.0 velocity=2.0 -> lower=-2.792526 upper=2.792526 effort=1000.0 velocity=1.0; origin xyz=0.079729 0.0 0.075 rpy=0 0 0 -> xyz=-0.075 0.0 0.0 rpy=0 -1.570796 0
- joint J5: limit lower=-2.094394 upper=2.094394 effort=1000.0 velocity=2.0 -> lower=-2.094394 upper=2.094394 effort=1000.0 velocity=1.0; origin xyz=0.130271 0.0 0.0 rpy=0 0 0 -> xyz=0.210 0.0 0.0 rpy=0 0 0
- joint J6: limit lower=-6.283185 upper=6.283185 effort=1000.0 velocity=2.0 -> lower=-6.283185 upper=6.283185 effort=1000.0 velocity=1.0

Commit message: added cublic spline trajectory to follow_joint_controller

File: robots/denso/vp6242_description/robot/vp6242.urdf (robot description, URDF)
Before this commit: robot vp6242, 7 links, 6 joints
Joints:
- joint J6: limit lower=-6.283185 upper=6.283185 effort=1000.0 velocity=1.0 -> lower=-3.141592 upper=3.141592 effort=1000.0 velocity=1.0

Commit message: updated follow joint controller

File: robots/denso/vp6242_description/robot/vp6242.urdf (robot description, URDF)
Before this commit: robot vp6242, 7 links, 6 joints
Joints:
- joint J6: limit lower=-3.141592 upper=3.141592 effort=1000.0 velocity=1.0 -> lower=-1.570796 upper=1.570796 effort=1000.0 velocity=1.0
