Commit message: - fixed joint velocity feedback problem - fixed prempted path problem - remove urdf (use xacro only)

File: robots/denso/vp6242_description/robot/vp6242.urdf.xacro (robot description, xacro)
@@ -11,5 +11,5 @@
   <xacro:property name="mesh_path" value="package://vp6242_description/robot" />
   <xacro:property name="mesh_scale" value="0.001 0.001 0.001" />
-  <xacro:property name="default_joint_velocity" value="1.0" />
+  <xacro:property name="default_joint_velocity" value="2.0" />
   <link name="base_link">
     <visual>

Commit message: update vp6242 xacro

File: robots/denso/vp6242_description/robot/vp6242.urdf.xacro (robot description, xacro)
@@ -11,5 +11,8 @@
   <xacro:property name="mesh_path" value="package://vp6242_description/robot" />
   <xacro:property name="mesh_scale" value="0.001 0.001 0.001" />
-  <xacro:property name="default_joint_velocity" value="2.0" />
+  <xacro:property name="default_joint_velocity" value="1.0" />
+  <xacro:property name="pi" value="3.1415926535897931" />
+  <xacro:property name="pi2" value="pi / 2.0" />
+  <xacro:property name="j6_limit" value="360" />
   <link name="base_link">
     <visual>
@@ -48,5 +51,5 @@
   <joint name="J1" type="revolute">
     <axis xyz="0 0 1"/>
-    <limit effort="1000.0" lower="-2.792526" upper="2.792526" velocity="${default_joint_velocity}"/>
+    <limit effort="1000.0" lower="${-(160.0/180.0) * pi}" upper="${(160.0/180.0) * pi}" velocity="${default_joint_velocity}"/>
     <origin rpy="0 0 0" xyz="0.0 0.0 0.155"/>
     <parent link="base_link"/>
@@ -70,5 +73,5 @@
   <joint name="J2" type="revolute">
     <axis xyz="0 1 0"/>
-    <limit effort="1000.0" lower="-2.094394" upper="2.094394" velocity="${default_joint_velocity}"/>
+    <limit effort="1000.0" lower="${-(120.0/180.0) * pi}" upper="${(120.0/180.0) * pi}" velocity="${default_joint_velocity}"/>
     <origin rpy="0 0 0" xyz="0.0 0.0 0.125"/>
     <parent link="link0"/>
@@ -92,5 +95,5 @@
  <joint name="J3" type="revolute">
     <axis xyz="0 1 0"/>
-    <limit effort="1000.0" lower="0.331612" upper="2.792526" velocity="${default_joint_velocity}"/>
+    <limit effort="1000.0" lower="${(19.0/180.0) * pi}" upper="${(160.0/180.0) * pi}" velocity="${default_joint_velocity}"/>
     <origin rpy="0 0 0" xyz="0.0 0.0 0.210"/>
     <parent link="link1"/>
@@ -114,5 +117,5 @@
   <joint name="J4" type="revolute">
     <axis xyz="1 0 0"/>
-    <limit effort="1000.0" lower="-2.792526" upper="2.792526" velocity="${default_joint_velocity}"/>
+    <limit effort="1000.0" lower="${-(160.0/180.0) * pi}" upper="${(160.0/180.0) * pi}" velocity="${default_joint_velocity}"/>
     <origin rpy="0 -1.570796 0" xyz="-0.075 0.0 0.0"/>
     <parent link="link2"/>
@@ -136,5 +139,5 @@
   <joint name="J5" type="revolute">
     <axis xyz="0 1 0"/>
-    <limit effort="1000.0" lower="-2.094394" upper="2.094394" velocity="${default_joint_velocity}"/>
+    <limit effort="1000.0" lower="${-(120.0/180.0) * pi}" upper="${(120.0/180.0) * pi}" velocity="${default_joint_velocity}"/>
     <origin rpy="0 0 0" xyz="0.210 0.0 0.0"/>
     <parent link="link3"/>
@@ -154,5 +157,5 @@
   <joint name="J6" type="revolute">
     <axis xyz="1 0 0"/>
-    <limit effort="1000.0" lower="-6.283185" upper="6.283185" velocity="${default_joint_velocity}"/>
+    <limit effort="1000.0" lower="${-(j6_limit/180.0) * pi}" upper="${(j6_limit/180.0) * pi}" velocity="${default_joint_velocity}"/>
     <origin rpy="0 0 0" xyz="0.07 0.0 0.0"/>
     <parent link="link4"/>

Commit message: updated

File: robots/denso/vp6242_description/robot/vp6242.urdf.xacro (robot description, xacro)
@@ -12,7 +12,7 @@
   <xacro:property name="mesh_scale" value="0.001 0.001 0.001" />
   <xacro:property name="default_joint_velocity" value="1.0" />
+  <xacro:property name="default_joint_effort" value="1.0" /> <!-- As acceleration limit -->
   <xacro:property name="pi" value="3.1415926535897931" />
   <xacro:property name="pi2" value="pi / 2.0" />
-  <xacro:property name="j6_limit" value="360" />
   <link name="base_link">
     <visual>
@@ -51,5 +51,5 @@
   <joint name="J1" type="revolute">
     <axis xyz="0 0 1"/>
-    <limit effort="1000.0" lower="${-(160.0/180.0) * pi}" upper="${(160.0/180.0) * pi}" velocity="${default_joint_velocity}"/>
+    <limit effort="${default_joint_effort}" lower="${-(160.0/180.0) * pi}" upper="${(160.0/180.0) * pi}" velocity="${default_joint_velocity}"/>
     <origin rpy="0 0 0" xyz="0.0 0.0 0.155"/>
     <parent link="base_link"/>
@@ -73,5 +73,5 @@
   <joint name="J2" type="revolute">
     <axis xyz="0 1 0"/>
-    <limit effort="1000.0" lower="${-(120.0/180.0) * pi}" upper="${(120.0/180.0) * pi}" velocity="${default_joint_velocity}"/>
+    <limit effort="${default_joint_effort}" lower="${-(120.0/180.0) * pi}" upper="${(120.0/180.0) * pi}" velocity="${default_joint_velocity}"/>
     <origin rpy="0 0 0" xyz="0.0 0.0 0.125"/>
     <parent link="link0"/>
@@ -95,5 +95,5 @@
  <joint name="J3" type="revolute">
     <axis xyz="0 1 0"/>
-    <limit effort="1000.0" lower="${(19.0/180.0) * pi}" upper="${(160.0/180.0) * pi}" velocity="${default_joint_velocity}"/>
+    <limit effort="${default_joint_effort}" lower="${(19.0/180.0) * pi}" upper="${(160.0/180.0) * pi}" velocity="${default_joint_velocity}"/>
     <origin rpy="0 0 0" xyz="0.0 0.0 0.210"/>
     <parent link="link1"/>
@@ -117,5 +117,5 @@
   <joint name="J4" type="revolute">
     <axis xyz="1 0 0"/>
-    <limit effort="1000.0" lower="${-(160.0/180.0) * pi}" upper="${(160.0/180.0) * pi}" velocity="${default_joint_velocity}"/>
+    <limit effort="${default_joint_effort}" lower="${-(160.0/180.0) * pi}" upper="${(160.0/180.0) * pi}" velocity="${default_joint_velocity}"/>
     <origin rpy="0 -1.570796 0" xyz="-0.075 0.0 0.0"/>
     <parent link="link2"/>
@@ -139,5 +139,5 @@
   <joint name="J5" type="revolute">
     <axis xyz="0 1 0"/>
-    <limit effort="1000.0" lower="${-(120.0/180.0) * pi}" upper="${(120.0/180.0) * pi}" velocity="${default_joint_velocity}"/>
+    <limit effort="${default_joint_effort}" lower="${-(120.0/180.0) * pi}" upper="${(120.0/180.0) * pi}" velocity="${default_joint_velocity}"/>
     <origin rpy="0 0 0" xyz="0.210 0.0 0.0"/>
     <parent link="link3"/>
@@ -157,5 +157,5 @@
   <joint name="J6" type="revolute">
     <axis xyz="1 0 0"/>
-    <limit effort="1000.0" lower="${-(j6_limit/180.0) * pi}" upper="${(j6_limit/180.0) * pi}" velocity="${default_joint_velocity}"/>
+    <limit effort="${default_joint_effort}" lower="${-(360/180.0) * pi}" upper="${(360/180.0) * pi}" velocity="${default_joint_velocity}"/>
     <origin rpy="0 0 0" xyz="0.07 0.0 0.0"/>
     <parent link="link4"/>

Commit message: updated

File: robots/denso/vp6242_description/robot/vp6242.urdf.xacro (robot description, xacro)
@@ -105,5 +105,5 @@
       <mesh filename="${mesh_path}/l3.stl" scale="${mesh_scale}"/>
     </geometry>
-    <origin rpy="-1.570796 3.141592 0" xyz="0.085 0 0.0"/>
+    <origin rpy="0 1.570796 1.570796" xyz="0 0 0.0"/>
 		<material name="link"/>
     </visual>
@@ -112,11 +112,11 @@
         <mesh filename="${mesh_path}/l3_collision.stl" scale="${mesh_scale}"/>
 	  	</geometry>
-      <origin rpy="-1.570796 3.141592 0" xyz="0.085 0 0"/>
+      <origin rpy="0 1.570796 1.570796" xyz="0 0 0.0"/>
     </collision>
   </link>
   <joint name="J4" type="revolute">
-    <axis xyz="1 0 0"/>
+    <axis xyz="0 0 1"/>
     <limit effort="${default_joint_effort}" lower="${-(160.0/180.0) * pi}" upper="${(160.0/180.0) * pi}" velocity="${default_joint_velocity}"/>
-    <origin rpy="0 -1.570796 0" xyz="-0.075 0.0 0.0"/>
+    <origin rpy="0 0 0" xyz="-0.075 0.0 0.085"/>
     <parent link="link2"/>
     <child link="link3"/>
@@ -127,5 +127,5 @@
   			<mesh filename="${mesh_path}/l4.stl" scale="${mesh_scale}"/>
       </geometry>
-    <xacro:mesh_origin/>
+    <origin rpy="0 1.570796 1.570796" xyz="0 0 0.0"/>
 	  <material name="link"/>
     </visual>
@@ -134,5 +134,5 @@
         <mesh filename="${mesh_path}/l4_collision.stl" scale="${mesh_scale}"/>
 	  	</geometry>
-      <xacro:mesh_origin/>
+      <origin rpy="0 1.570796 1.570796" xyz="0 0 0.0"/>
     </collision>
   </link>
@@ -140,5 +140,5 @@
     <axis xyz="0 1 0"/>
     <limit effort="${default_joint_effort}" lower="${-(120.0/180.0) * pi}" upper="${(120.0/180.0) * pi}" velocity="${default_joint_velocity}"/>
-    <origin rpy="0 0 0" xyz="0.210 0.0 0.0"/>
+    <origin rpy="0 0 0" xyz="0.0 0.0 0.135"/>
     <parent link="link3"/>
     <child link="link4"/>
@@ -147,7 +147,7 @@
   <visual>
     <geometry>
-      <cylinder length="0.010" radius="0.021"/>
+      <cylinder length="0.01" radius="0.0205"/>
     </geometry>
-    <origin rpy="0 1.570796 0" xyz="-0.004 0.0 0.0"/>
+    <origin rpy="0 0 0" xyz="0.0 0.0 0.0"/>
     <material name="plate">
       <color rgba="0.1 0.1 0.1 0.8"/>
@@ -156,7 +156,7 @@
   </link>
   <joint name="J6" type="revolute">
-    <axis xyz="1 0 0"/>
+    <axis xyz="0 0 1"/>
     <limit effort="${default_joint_effort}" lower="${-(360/180.0) * pi}" upper="${(360/180.0) * pi}" velocity="${default_joint_velocity}"/>
-    <origin rpy="0 0 0" xyz="0.07 0.0 0.0"/>
+    <origin rpy="0 0 0" xyz="0.0 0.0 0.07"/>
     <parent link="link4"/>
     <child link="link5"/>

Commit message: fixed ik fast plugin bug  - it was reporting the first found solution not the closest solution before fixed

File: robots/denso/vp6242_description/robot/vp6242.urdf.xacro (robot description, xacro)
@@ -105,5 +105,5 @@
       <mesh filename="${mesh_path}/l3.stl" scale="${mesh_scale}"/>
     </geometry>
-    <origin rpy="0 1.570796 1.570796" xyz="0 0 0.0"/>
+    <origin rpy="0 1.570796 1.570796" xyz="0 0 0.085"/>
 		<material name="link"/>
     </visual>
@@ -112,5 +112,5 @@
         <mesh filename="${mesh_path}/l3_collision.stl" scale="${mesh_scale}"/>
 	  	</geometry>
-      <origin rpy="0 1.570796 1.570796" xyz="0 0 0.0"/>
+      <origin rpy="0 1.570796 1.570796" xyz="0 0 0.085"/>
     </collision>
   </link>
@@ -118,5 +118,5 @@
     <axis xyz="0 0 1"/>
     <limit effort="${default_joint_effort}" lower="${-(160.0/180.0) * pi}" upper="${(160.0/180.0) * pi}" velocity="${default_joint_velocity}"/>
-    <origin rpy="0 0 0" xyz="-0.075 0.0 0.085"/>
+    <origin rpy="0 0 0" xyz="-0.075 0.0 0.0"/>
     <parent link="link2"/>
     <child link="link3"/>
@@ -140,5 +140,5 @@
     <axis xyz="0 1 0"/>
     <limit effort="${default_joint_effort}" lower="${-(120.0/180.0) * pi}" upper="${(120.0/180.0) * pi}" velocity="${default_joint_velocity}"/>
-    <origin rpy="0 0 0" xyz="0.0 0.0 0.135"/>
+    <origin rpy="0 0 0" xyz="0.0 0.0 0.210"/>
     <parent link="link3"/>
     <child link="link4"/>

Commit message: updated vp6242 xacro

File: robots/denso/vp6242_description/robot/vp6242.urdf.xacro (robot description, xacro)
@@ -149,5 +149,5 @@
       <cylinder length="0.01" radius="0.0205"/>
     </geometry>
-    <origin rpy="0 0 0" xyz="0.0 0.0 0.0"/>
+    <origin rpy="0 -1.570796 0" xyz="0.0 0.0 0.0"/>
     <material name="plate">
       <color rgba="0.1 0.1 0.1 0.8"/>
@@ -156,7 +156,7 @@
   </link>
   <joint name="J6" type="revolute">
-    <axis xyz="0 0 1"/>
+    <axis xyz="1 0 0"/>
     <limit effort="${default_joint_effort}" lower="${-(360/180.0) * pi}" upper="${(360/180.0) * pi}" velocity="${default_joint_velocity}"/>
-    <origin rpy="0 0 0" xyz="0.0 0.0 0.07"/>
+    <origin rpy="0 -1.570796 0" xyz="0.0 0.0 0.07"/>
     <parent link="link4"/>
     <child link="link5"/>

Commit message: changed joint acceleration to 4.0

File: robots/denso/vp6242_description/robot/vp6242.urdf.xacro (robot description, xacro)
@@ -12,5 +12,5 @@
   <xacro:property name="mesh_scale" value="0.001 0.001 0.001" />
   <xacro:property name="default_joint_velocity" value="1.0" />
-  <xacro:property name="default_joint_effort" value="1.0" /> <!-- As acceleration limit -->
+  <xacro:property name="default_joint_effort" value="4.0" /> <!-- As acceleration limit -->
   <xacro:property name="pi" value="3.1415926535897931" />
   <xacro:property name="pi2" value="pi / 2.0" />

Commit message: separted launch file (sensors/motion)

File: robots/denso/vp6242_description/robot/vp6242.urdf.xacro (robot description, xacro)
@@ -12,5 +12,5 @@
   <xacro:property name="mesh_scale" value="0.001 0.001 0.001" />
   <xacro:property name="default_joint_velocity" value="1.0" />
-  <xacro:property name="default_joint_effort" value="4.0" /> <!-- As acceleration limit -->
+  <xacro:property name="default_joint_effort" value="1.0" /> <!-- As acceleration limit -->
   <xacro:property name="pi" value="3.1415926535897931" />
   <xacro:property name="pi2" value="pi / 2.0" />

Commit message: change mesh to dae

File: robots/denso/vp6242_description/robot/vp6242.urdf.xacro (robot description, xacro)
@@ -18,5 +18,5 @@
     <visual>
 	  <geometry>
-	    <mesh filename="${mesh_path}/base.stl" scale="${mesh_scale}"/>
+	    <mesh filename="${mesh_path}/base.dae" scale="${mesh_scale}"/>
 	  </geometry>
     <xacro:mesh_origin/>
@@ -27,5 +27,5 @@
     <collision>
 	  	<geometry>
-  	    <mesh filename="${mesh_path}/base_collision.stl" scale="${mesh_scale}"/>
+  	    <mesh filename="${mesh_path}/base_collision.dae" scale="${mesh_scale}"/>
 	  	</geometry>
       <xacro:mesh_origin/>
@@ -35,5 +35,5 @@
     <visual>
       <geometry>
-   	    <mesh filename="${mesh_path}/l0.stl" scale="${mesh_scale}"/>
+   	    <mesh filename="${mesh_path}/l0.dae" scale="${mesh_scale}"/>
       </geometry>
       <xacro:mesh_origin/>
@@ -44,5 +44,5 @@
     <collision>
 	  	<geometry>
-        <mesh filename="${mesh_path}/l0_collision.stl" scale="${mesh_scale}"/>
+        <mesh filename="${mesh_path}/l0_collision.dae" scale="${mesh_scale}"/>
 	  	</geometry>
       <xacro:mesh_origin/>
@@ -59,5 +59,5 @@
     <visual>
       <geometry>
-   	    <mesh filename="${mesh_path}/l1.stl" scale="${mesh_scale}"/>
+   	    <mesh filename="${mesh_path}/l1.dae" scale="${mesh_scale}"/>
       </geometry>
       <xacro:mesh_origin/>
@@ -66,5 +66,5 @@
     <collision>
      	<geometry>
-        <mesh filename="${mesh_path}/l1_collision.stl" scale="${mesh_scale}"/>
+        <mesh filename="${mesh_path}/l1_collision.dae" scale="${mesh_scale}"/>
 	  	</geometry>
       <xacro:mesh_origin/>
@@ -81,5 +81,5 @@
     <visual>
       <geometry>
-   	    <mesh filename="${mesh_path}/l2.stl" scale="${mesh_scale}"/>
+   	    <mesh filename="${mesh_path}/l2.dae" scale="${mesh_scale}"/>
       </geometry>
       <origin rpy="-1.570796 1.570796 0" xyz="0 0 0"/>
@@ -88,5 +88,5 @@
     <collision>
       <geometry>
-        <mesh filename="${mesh_path}/l2_collision.stl" scale="${mesh_scale}"/>
+        <mesh filename="${mesh_path}/l2_collision.dae" scale="${mesh_scale}"/>
 	  	</geometry>
       <origin rpy="-1.570796 1.570796 0" xyz="0 0 0"/>
@@ -103,5 +103,5 @@
     <visual>
     <geometry>
-      <mesh filename="${mesh_path}/l3.stl" scale="${mesh_scale}"/>
+      <mesh filename="${mesh_path}/l3.dae" scale="${mesh_scale}"/>
     </geometry>
     <origin rpy="0 1.570796 1.570796" xyz="0 0 0.085"/>
@@ -110,5 +110,5 @@
     <collision>
 	  	<geometry>
-        <mesh filename="${mesh_path}/l3_collision.stl" scale="${mesh_scale}"/>
+        <mesh filename="${mesh_path}/l3_collision.dae" scale="${mesh_scale}"/>
 	  	</geometry>
       <origin rpy="0 1.570796 1.570796" xyz="0 0 0.085"/>
@@ -125,5 +125,5 @@
     <visual>
       <geometry>
-  			<mesh filename="${mesh_path}/l4.stl" scale="${mesh_scale}"/>
+  			<mesh filename="${mesh_path}/l4.dae" scale="${mesh_scale}"/>
       </geometry>
     <origin rpy="0 1.570796 1.570796" xyz="0 0 0.0"/>
@@ -132,5 +132,5 @@
     <collision>
 	  	<geometry>
-        <mesh filename="${mesh_path}/l4_collision.stl" scale="${mesh_scale}"/>
+        <mesh filename="${mesh_path}/l4_collision.dae" scale="${mesh_scale}"/>
 	  	</geometry>
       <origin rpy="0 1.570796 1.570796" xyz="0 0 0.0"/>
