Commit message: add vp6242 moveit

File: robots/industrial/denso/denso_common/urdf/vp6242_macro.xacro (robot description, xacro)
@@ -192,5 +192,5 @@
                 velocity="${default_joint_velocity}"/>
         </joint>
-        <joint name="J6" type="revolute">
+        <joint name="${prefix}joint6" type="revolute">
             <origin rpy="0 -1.570796 0" xyz="0.0 0.0 0.07"/>
             <parent link="link5"/>

Commit message: constructing controller

File: robots/industrial/denso/denso_common/urdf/vp6242_macro.xacro (robot description, xacro)
@@ -36,4 +36,5 @@
     <xacro:macro name="vp6242" params="prefix">
         <!-- Link lisk -->
+        <link name="${prefix}base"/>
         <link name="${prefix}base_link">
             <xacro:default_inertial mass="10"/>
@@ -139,4 +140,9 @@
         <link name="${prefix}tool0"/>
         <!-- Joint lisk -->
+        <joint name="${prefix}base-base_link" type="fixed">
+			<parent link="${prefix}base"/>
+			<child link="${prefix}base_link"/>
+			<origin xyz="0 0 0" rpy="0 0 0"/>
+		</joint>
         <joint name="${prefix}joint1" type="revolute">
             <origin rpy="0 0 0" xyz="0.0 0.0 0.155"/>
@@ -158,6 +164,6 @@
         <joint name="${prefix}joint2" type="revolute">
             <origin rpy="0 0 0" xyz="0.0 0.0 0.125"/>
-            <parent link="link1"/>
-            <child link="link2"/>
+            <parent link="${prefix}link1"/>
+            <child link="${prefix}link2"/>
             <axis xyz="0 1 0"/>
             <limit
@@ -175,6 +181,6 @@
         <joint name="${prefix}joint3" type="revolute">
             <origin rpy="0 0 0" xyz="0.0 0.0 0.210"/>
-            <parent link="link2"/>
-            <child link="link3"/>
+            <parent link="${prefix}link2"/>
+            <child link="${prefix}link3"/>
             <axis xyz="0 1 0"/>
             <limit
@@ -186,6 +192,6 @@
         <joint name="${prefix}joint4" type="revolute">
             <origin rpy="0 0 0" xyz="-0.075 0.0 0.0"/>
-            <parent link="link3"/>
-            <child link="link4"/>
+            <parent link="${prefix}link3"/>
+            <child link="${prefix}link4"/>
             <axis xyz="0 0 1"/>
             <limit
@@ -197,6 +203,6 @@
         <joint name="${prefix}joint5" type="revolute">
             <origin rpy="0 0 0" xyz="0.0 0.0 0.210"/>
-            <parent link="link4"/>
-            <child link="link5"/>
+            <parent link="${prefix}link4"/>
+            <child link="${prefix}link5"/>
             <axis xyz="0 1 0"/>
             <limit
@@ -208,6 +214,6 @@
         <joint name="${prefix}joint6" type="revolute">
             <origin rpy="0 -1.570796 0" xyz="0.0 0.0 0.07"/>
-            <parent link="link5"/>
-            <child link="link6"/>
+            <parent link="${prefix}link5"/>
+            <child link="${prefix}link6"/>
             <axis xyz="1 0 0"/>
             <limit
@@ -218,6 +224,6 @@
         </joint>
         <joint name="${prefix}joint6-tool0" type="fixed">
-			<parent link="link6"/>
-			<child link="tool0"/>
+			<parent link="${prefix}link6"/>
+			<child link="${prefix}tool0"/>
 			<origin xyz="0 0 0" rpy="0 0 0"/>
 		</joint>
