Commit message: add controller manager (copy from ros control)

File: robots/industrial/denso/denso_common/urdf/vp6242.urdf (robot description, URDF)
Before this commit: robot vp6242, 8 links, 7 joints
Links:
- link base_link: mass None -> 10
- link link1: mass None -> 1
- link link2: mass None -> 1
- link link3: mass None -> 1
- link link4: mass None -> 1
- link link5: mass None -> 1

File: robots/industrial/denso/denso_common/urdf/vp6242_macro.xacro (robot description, xacro)
@@ -26,7 +26,16 @@
     <xacro:property name="joint6_max" value="6.283185307"/>
     <xacro:property name="joint6_min" value="-6.283185307"/>
+    <xacro:macro name="default_inertial" params="mass">
+        <inertial>
+            <mass value="${mass}" />
+            <inertia ixx="1.0" ixy="0.0" ixz="0.0"
+                     iyy="1.0" iyz="0.0"
+                     izz="1.0" />
+        </inertial>
+    </xacro:macro>
     <xacro:macro name="vp6242" params="prefix">
         <!-- Link lisk -->
         <link name="${prefix}base_link">
+            <xacro:default_inertial mass="10"/>
             <visual>
 	            <geometry>
@@ -43,4 +52,5 @@
         </link>
         <link name="${prefix}link1">
+            <xacro:default_inertial mass="1"/>
             <visual>
                 <geometry>
@@ -57,4 +67,5 @@
         </link>
         <link name="${prefix}link2">
+            <xacro:default_inertial mass="1"/>
             <visual>
                 <geometry>
@@ -71,4 +82,5 @@
         </link>
         <link name="${prefix}link3">
+            <xacro:default_inertial mass="1"/>
             <visual>
                 <geometry>
@@ -85,4 +97,5 @@
         </link>
         <link name="${prefix}link4">
+            <xacro:default_inertial mass="1"/>
             <visual>
                 <geometry>
@@ -99,4 +112,5 @@
         </link>
         <link name="${prefix}link5">
+            <xacro:default_inertial mass="1"/>
             <visual>
                 <geometry>

Commit message: moveit is now working mix codes from industial, pr2, ros_control

File: robots/industrial/denso/denso_common/urdf/vp6242.urdf (robot description, URDF)
Before this commit: robot vp6242, 8 links, 7 joints
Links:
- added link base
Joints:
- added joint base-base_link: type fixed, parent base, child base_link, origin xyz=0 0 0 rpy=0 0 0
